File: keybored.brd (EAGLE design)
At the start: 245.1 x 100 mm, 130 parts

Commit message: preliminary layout
Parts:
- moved UP 381.6 mm to (234.9, 23.5)
- moved RIGHT 364.0 mm to (250.2, 8.26)
- moved DOWN 357.2 mm to (234.9, 8.26)
- moved D41 354.5 mm to (231.8, 29.2), flipped to the bottom
- moved RSHIFT 337.7 mm to (210.2, 23.5)
- moved D65 324.3 mm to (217.2, 52.7), flipped to the bottom
- moved D36 322.7 mm to (216.5, 14.0), flipped to the bottom
- moved R_CMD 322.1 mm to (174.0, 8.26)
- moved D20 322.0 mm to (170.8, 14.0), flipped to the bottom
- moved D49 313.7 mm to (147.3, 29.2), flipped to the bottom
- moved D48 310.5 mm to (154.9, 44.5), flipped to the bottom
- moved D51 301.0 mm to (247.0, 14.0), flipped to the bottom
- moved D64 301.0 mm to (204.5, 74.9), flipped to the bottom
- moved D60 299.6 mm to (207.0, 29.2), flipped to the bottom
- moved [ 297.4 mm to (184.8, 54.0)
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Connections:
- net COL10: now also D20.P$2; no longer D50.P$2
- net COL11: no longer D51.P$2
- net COL12: now also D35.P$2
- net COL13: now also D36.P$2
- net COL14: now also D41.P$2, D50.P$2, D51.P$2
- net COL5: no longer D25.P$2
- net COL6: no longer D20.P$2
- net COL7: now also D25.P$2; no longer D35.P$2
- net COL8: no longer D36.P$2
- net COL9: no longer D41.P$2
Routing:
- net ROW5: track 0.00 -> 264.6 mm
- net ROW3: track 0.00 -> 212.6 mm
- net ROW4: track 0.00 -> 204.8 mm
- net ROW1: track 0.00 -> 204.6 mm
- net ROW2: track 0.00 -> 192.7 mm
- net COL14: track 0.00 -> 93.7 mm
- net COL10: track 0.00 -> 90.1 mm
- net COL13: track 0.00 -> 80.4 mm
- net COL7: track 0.00 -> 79.9 mm
- net COL12: track 0.00 -> 79.2 mm
- net COL4: track 0.00 -> 75.1 mm
- net COL3: track 0.00 -> 75.1 mm
- net COL2: track 0.00 -> 73.9 mm
- net COL1: track 0.00 -> 73.6 mm
- net COL8: track 0.00 -> 58.2 mm
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Other:
- board size 245.1 x 100 mm -> 260.4 x 78.1 mm
