File: keybored.sch (EAGLE design)
At the start: 130 parts

Commit message: preliminary layout
Connections:
- net COL10: now also D20.P$2; no longer D50.P$2
- net COL11: no longer D51.P$2
- net COL12: now also D35.P$2
- net COL13: now also D36.P$2
- net COL14: now also D41.P$2, D50.P$2, D51.P$2
- net COL5: no longer D25.P$2
- net COL6: no longer D20.P$2
- net COL7: now also D25.P$2; no longer D35.P$2
- net COL8: no longer D36.P$2
- net COL9: no longer D41.P$2
Other:
- moved on the sheet: DOWN, LEFT, RIGHT, R_CMD, R_OPTION, SPACE, UP
